File: plaqchek_power/plaqchek_power.kicad_sch (KiCad schematic)
At the start: 11 parts, among them J1 Conn_01x04, J2 Conn_01x04, J4 Conn_01x03, J5 Barrel_Jack, U16 LDK320AM-R

Commit message: finish schematic
Parts:
- removed C43, C44: 1uF, symbol Device:C_Small
- removed J1: Conn_01x04, symbol Connector_Generic:Conn_01x04
- removed R29: 350kR, symbol Device:R_Small_US
- removed R30: 100kR, symbol Device:R_Small_US
- removed U16: LDK320AM-R, symbol plaqchek_mlb:LDK320AM-R
- added D2 (x2), D4, D5: RED, symbol Device:LED
- added J1: Conn_01x05, symbol Connector_Generic:Conn_01x05
- added R31: 2.5kR, symbol Device:R_Small_US
- added R31, R34: 250R, symbol Device:R_Small_US
- added R33: 75R, symbol Device:R_Small_US
- added TP9: TestPoint, symbol Connector:TestPoint
Connections:
- net +12V: now also TP9.1
- net +3V3: now also J1.3 (Pin_3), R33.1
- net +6V: now also J1.2 (Pin_2), R31.1
- net -6V5: now also D5.1 (K), J1.4 (Pin_4)
- net GND: now also D2.1 (K), D2.1 (K), D4.1 (K), J1.5 (Pin_5), R34.1
- new net: D2.2 (A), R31.2 (x2)
- new net: D4.2 (A), R33.2
- new net: D5.2 (A), R34.2
- new net SIPM_BIAS_OUT: J1.1 (Pin_1), R31.1
Other:
- note added: "12V 2A (24W)"
- note added: "FOR VF=1.9V, MAX IF=20mA"
- note removed: "12V 2A (24V)"
- note removed: "Max dropout V = 350mV"
- note removed: "Vadj = 1.185 typ Vo = Vadj * (1 + R1 / R2)"
- note removed: "enables photodetection (turns off bias)"

Commit message: more footprints and some value fixes
Parts:
- C13, C14: footprint (none) -> Capacitor_SMD:C_0603_1608Metric_Pad1.08x0.95mm_HandSolder
Changed lines of the file:
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@@
       (effects (font (size 1.27 1.27)) (justify left))
     )
-    (property "Footprint" "" (at 46.99 29.21 0)
+    (property "Footprint" "Capacitor_SMD:C_0603_1608Metric_Pad1.08x0.95mm_HandSolder" (at 46.99 29.21 0)
       (effects (font (size 1.27 1.27)) hide)
     )
@@
       (effects (font (size 1.27 1.27)) (justify left))
     )
-    (property "Footprint" "" (at 60.96 29.21 0)
+    (property "Footprint" "Capacitor_SMD:C_0603_1608Metric_Pad1.08x0.95mm_HandSolder" (at 60.96 29.21 0)
       (effects (font (size 1.27 1.27)) hide)
     )

Commit message: finish main logic board PCB routing
Parts:
- D2, D4, D5: footprint (none) -> Diode_SMD:D_0805_2012Metric_Pad1.15x1.40mm_HandSolder
- J1: footprint (none) -> Connector_PinHeader_2.54mm:PinHeader_1x05_P2.54mm_Vertical
- J2: footprint (none) -> Connector_PinHeader_2.54mm:PinHeader_1x04_P2.54mm_Vertical
- J4: footprint (none) -> Connector_PinHeader_2.54mm:PinHeader_1x03_P2.54mm_Vertical
- J5: footprint (none) -> Connector_BarrelJack:BarrelJack_Horizontal
- R31, R33, R34: footprint (none) -> Resistor_SMD:R_0603_1608Metric_Pad0.98x0.95mm_HandSolder
Changed lines of the file:
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@@
       (effects (font (size 1.27 1.27)))
     )
-    (property "Footprint" "" (at 106.68 160.02 0)
+    (property "Footprint" "Resistor_SMD:R_0603_1608Metric_Pad0.98x0.95mm_HandSolder" (at 106.68 160.02 0)
       (effects (font (size 1.27 1.27)) hide)
     )
@@
       (effects (font (size 1.27 1.27)))
     )
-    (property "Footprint" "" (at 256.54 69.85 0)
+    (property "Footprint" "Connector_PinHeader_2.54mm:PinHeader_1x03_P2.54mm_Vertical" (at 256.54 69.85 0)
       (effects (font (size 1.27 1.27)) hide)
     )
@@
       (effects (font (size 1.27 1.27)) (justify right))
     )
-    (property "Footprint" "" (at 80.01 172.72 0)
+    (property "Footprint" "Diode_SMD:D_0805_2012Metric_Pad1.15x1.40mm_HandSolder" (at 80.01 172.72 0)
       (effects (font (size 1.27 1.27)) hide)
     )
@@
       (effects (font (size 1.27 1.27)))
     )
-    (property "Footprint" "" (at 248.92 35.56 0)
+    (property "Footprint" "Connector_PinHeader_2.54mm:PinHeader_1x04_P2.54mm_Vertical" (at 248.92 35.56 0)
       (effects (font (size 1.27 1.27)) hide)
     )
@@
       (effects (font (size 1.27 1.27)))
     )
-    (property "Footprint" "" (at 80.01 165.1 0)
+    (property "Footprint" "Resistor_SMD:R_0603_1608Metric_Pad0.98x0.95mm_HandSolder" (at 80.01 165.1 0)
       (effects (font (size 1.27 1.27)) hide)
     )
@@
       (effects (font (size 1.27 1.27)) (justify right))
     )
-    (property "Footprint" "" (at 36.83 168.91 0)
+    (property "Footprint" "Diode_SMD:D_0805_2012Metric_Pad1.15x1.40mm_HandSolder" (at 36.83 168.91 0)
       (effects (font (size 1.27 1.27)) hide)
     )
@@
       (effects (font (size 1.27 1.27)))
     )
-    (property "Footprint" "" (at 60.96 160.02 0)
+    (property "Footprint" "Resistor_SMD:R_0603_1608Metric_Pad0.98x0.95mm_HandSolder" (at 60.96 160.02 0)
       (effects (font (size 1.27 1.27)) hide)
     )
@@
       (effects (font (size 1.27 1.27)))
     )
-    (property "Footprint" "" (at 25.4 28.956 0)
+    (property "Footprint" "Connector_BarrelJack:BarrelJack_Horizontal" (at 25.4 28.956 0)
       (effects (font (size 1.27 1.27)) hide)
     )
@@
       (effects (font (size 1.27 1.27)) (justify right))
     )
-    (property "Footprint" "" (at 60.96 170.18 0)
+    (property "Footprint" "Diode_SMD:D_0805_2012Metric_Pad1.15x1.40mm_HandSolder" (at 60.96 170.18 0)
       (effects (font (size 1.27 1.27)) hide)
     )
@@
       (effects (font (size 1.27 1.27)) (justify right))
     )
-    (property "Footprint" "" (at 106.68 170.18 0)
+    (property "Footprint" "Diode_SMD:D_0805_2012Metric_Pad1.15x1.40mm_HandSolder" (at 106.68 170.18 0)
       (effects (font (size 1.27 1.27)) hide)
     )
@@
       (effects (font (size 1.27 1.27)))
     )
-    (property "Footprint" "" (at 245.11 105.41 0)
+    (property "Footprint" "Connector_PinHeader_2.54mm:PinHeader_1x05_P2.54mm_Vertical" (at 245.11 105.41 0)
       (effects (font (size 1.27 1.27)) hide)
     )
@@
       (effects (font (size 1.27 1.27)))
     )
-    (property "Footprint" "" (at 36.83 158.75 0)
-      (effects (font (size 1.27 1.27)) hide)
-    )
+    (property "Footprint" "Resistor_SMD:R_0603_1608Metric_Pad0.98x0.95mm_HandSolder" (at 36.83 158.75 0)
+      (effects (font (size 1.27 1.27)) hide)
+    )

Commit message: finish power board routing, sensing board routing
Parts:
- removed J5: Barrel_Jack, Connector_BarrelJack:BarrelJack_Horizontal, symbol Connector:Barrel_Jack
- added H1, H2, H3, H4: MountingHole_Pad, MountingHole:MountingHole_3.2mm_M3_Pad, symbol Mechanical:MountingHole_Pad
- added J3: Barrel_Jack_Switch, Connector_BarrelJack:BarrelJack_Horizontal, symbol Connector:Barrel_Jack_Switch
- added R1 (x4): 0R, Resistor_SMD:R_0603_1608Metric_Pad0.98x0.95mm_HandSolder, symbol Device:R_Small_US
- added TP10, TP11, TP12, TP13, TP14, TP15, TP16, TP17: TestPoint, TestPoint:TestPoint_Pad_D1.0mm, symbol Connector:TestPoint
- TP9: footprint (none) -> TestPoint:TestPoint_Pad_D1.0mm
Connections:
- net +12V: now also J3.1
- net GND: now also J3.2, J3.3, R1.2, R1.2, R1.2, R1.2, TP10.1, TP11.1, TP12.1, TP13.1, TP14.1, TP15.1, TP16.1, TP17.1
- new net: H2.1, R1.1
- new net: H1.1, R1.1
- new net: H3.1, R1.1
- new net: H4.1, R1.1
