File: plaqchek_power/plaqcheq_power_sipm.kicad_sch (KiCad schematic)
At the start: 25 parts, among them U1 LM5157

Commit message: finish power board routing, sensing board routing
Parts:
- C52: footprint Capacitor_SMD:C_0805_2012Metric_Pad1.18x1.45mm_HandSolder -> Capacitor_SMD:C_0603_1608Metric_Pad1.08x0.95mm_HandSolder
- TP3, TP4: footprint (none) -> TestPoint:TestPoint_Pad_D1.0mm
Connections:
- net PD_BOOST_OUT is gone; now on net VOUT_SIPM: R45.2
- net VB_SIPM: now reaches C47.1, C48.2, L4.1, R23.1, R43.2, U1.3 (BIAS)
- net VOUT_SIPM: now reaches C53.2, C54.2, D2.1 (K), R23.2, R37.1, TP3.1
- net VCC_SIPM: now reaches R42.2, U1.2 (VCC)
- net RT_SIPM: now reaches R46.2, U1.5 (RT)
- net EN_SIPM_R: now reaches R23.1, U1.6 (EN/UVLO/SYNC)
- net COMP_SIPM: now reaches C50.1, C51.2, U1.8 (COMP)
- net SS_SIPM: now reaches C52.2, U1.10 (SS)
- net MODE_SIPM: now reaches R40.1, U1.11 (MODE)
- net FB_SIPM_OUT: now reaches R37.2, R38.1, U1.9 (FB)
- net PD_BOOST_PGOOD renamed PD_BOOST_PG
Other:
- note added: "Iout max = 50mA"
- note removed: "Iout max = 500mA"
- moved on the sheet: R40
Changed lines of the file:
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@@
   (junction (at 149.86 129.54) (diameter 0) (color 0 0 0 0)
   )
-  (junction (at 181.61 129.54) (diameter 0) (color 0 0 0 0)
-  )
   (junction (at 205.74 96.52) (diameter 0) (color 0 0 0 0)
   )
@@
   )
   (junction (at 66.04 90.17) (diameter 0) (color 0 0 0 0)
+  )
+  (junction (at 184.912 129.54) (diameter 0) (color 0 0 0 0)
   )
   (junction (at 49.53 54.61) (diameter 0) (color 0 0 0 0)
@@
     (stroke (width 0) (type default))
   )
-  (wire (pts (xy 181.61 129.54) (xy 158.75 129.54))
+  (wire (pts (xy 158.75 129.54) (xy 184.912 129.54))
     (stroke (width 0) (type default))
   )
@@
     (stroke (width 0) (type default))
   )
-  (wire (pts (xy 205.74 129.54) (xy 181.61 129.54))
-    (stroke (width 0) (type default))
-  )
-  (wire (pts (xy 181.61 115.57) (xy 181.61 129.54))
+  (wire (pts (xy 205.74 129.54) (xy 184.912 129.54))
+    (stroke (width 0) (type default))
+  )
+  (wire (pts (xy 184.912 115.57) (xy 184.912 129.54))
     (stroke (width 0) (type default))
   )
@@
     (stroke (width 0) (type default))
   )
-  (wire (pts (xy 166.37 115.57) (xy 170.18 115.57))
+  (wire (pts (xy 166.37 115.57) (xy 178.562 115.57))
     (stroke (width 0) (type default))
   )
@@
     (stroke (width 0) (type default))
   )
-  (wire (pts (xy 175.26 115.57) (xy 181.61 115.57))
+  (wire (pts (xy 183.642 115.57) (xy 184.912 115.57))
     (stroke (width 0) (type default))
   )
@@
     (effects (font (size 5 5) (thickness 1) bold) (justify left bottom))
   )
-  (text "Iout max = 500mA\n" (at 261.62 58.42 0)
+  (text "Iout max = 50mA\n" (at 261.62 58.42 0)
     (effects (font (size 1.27 1.27)) (justify left bottom))
   )
@@
     (effects (font (size 1.27 1.27)) (justify left bottom))
   )
-  (label "PD_BOOST_PGOOD" (at 203.2 109.22 180) (fields_autoplaced)
+  (label "COMP_SIPM" (at 118.618 109.22 0) (fields_autoplaced)
+    (effects (font (size 1.27 1.27)) (justify left bottom))
+  )
+  (label "VCC_SIPM" (at 149.86 75.438 90) (fields_autoplaced)
+    (effects (font (size 1.27 1.27)) (justify left bottom))
+  )
+  (label "EN_SIPM" (at 70.612 90.17 0) (fields_autoplaced)
+    (effects (font (size 1.27 1.27)) (justify left bottom))
+  )
+  (label "VOUT_SIPM" (at 213.36 54.61 0) (fields_autoplaced)
+    (effects (font (size 1.27 1.27)) (justify left bottom))
+  )
+  (label "PD_BOOST_PG" (at 203.2 109.22 180) (fields_autoplaced)
     (effects (font (size 1.27 1.27)) (justify right bottom))
   )
-  (label "PD_BOOST_OUT" (at 166.37 100.33 0) (fields_autoplaced)
+  (label "FB_SIPM_OUT" (at 171.704 96.52 0) (fields_autoplaced)
+    (effects (font (size 1.27 1.27)) (justify left bottom))
+  )
+  (label "MODE_SIPM" (at 167.894 115.57 0) (fields_autoplaced)
+    (effects (font (size 1.27 1.27)) (justify left bottom))
+  )
+  (label "VB_SIPM" (at 94.742 54.61 0) (fields_autoplaced)
+    (effects (font (size 1.27 1.27)) (justify left bottom))
+  )
+  (label "RT_SIPM" (at 98.552 96.52 0) (fields_autoplaced)
+    (effects (font (size 1.27 1.27)) (justify left bottom))
+  )
+  (label "VOUT_SIPM" (at 169.926 100.33 0) (fields_autoplaced)
+    (effects (font (size 1.27 1.27)) (justify left bottom))
+  )
+  (label "SS_SIPM" (at 106.934 102.87 0) (fields_autoplaced)
+    (effects (font (size 1.27 1.27)) (justify left bottom))
+  )
+  (label "EN_SIPM_R" (at 98.298 90.17 0) (fields_autoplaced)
     (effects (font (size 1.27 1.27)) (justify left bottom))
   )
@@
       (effects (font (size 1.27 1.27)) (justify left))
     )
-    (property "Footprint" "" (at 248.92 49.53 0)
+    (property "Footprint" "TestPoint:TestPoint_Pad_D1.0mm" (at 248.92 49.53 0)
       (effects (font (size 1.27 1.27)) hide)
     )
@@
       (effects (font (size 1.27 1.27)) (justify left))
     )
-    (property "Footprint" "" (at 262.89 49.53 0)
+    (property "Footprint" "TestPoint:TestPoint_Pad_D1.0mm" (at 262.89 49.53 0)
       (effects (font (size 1.27 1.27)) hide)
     )
@@
       (effects (font (size 1.27 1.27)) (justify right))
     )
-    (property "Footprint" "Capacitor_SMD:C_0805_2012Metric_Pad1.18x1.45mm_HandSolder" (at 97.79 114.3 0)
+    (property "Footprint" "Capacitor_SMD:C_0603_1608Metric_Pad1.08x0.95mm_HandSolder" (at 97.79 114.3 0)
       (effects (font (size 1.27 1.27)) hide)
     )
@@
     )
   )
-  (symbol (lib_id "Device:R_Small_US") (at 172.72 115.57 90) (unit 1)
+  (symbol (lib_id "Device:R_Small_US") (at 181.102 115.57 90) (unit 1)
     (in_bom yes) (on_board yes) (dnp no) (fields_autoplaced)
-    (property "Reference" "R40" (at 172.72 111.125 90)
-      (effects (font (size 1.27 1.27)))
-    )
-    (property "Value" "0R" (at 172.72 113.665 90)
-      (effects (font (size 1.27 1.27)))
-    )
-    (property "Footprint" "Resistor_SMD:R_0603_1608Metric_Pad0.98x0.95mm_HandSolder" (at 172.72 115.57 0)
-      (effects (font (size 1.27 1.27)) hide)
-    )
-    (property "Datasheet" "~" (at 172.72 115.57 0)
-      (effects (font (size 1.27 1.27)) hide)
-    )
+    (property "Reference" "R40" (at 181.102 111.125 90)
+      (effects (font (size 1.27 1.27)))
+    )
+    (property "Value" "0R" (at 181.102 113.665 90)
+      (effects (font (size 1.27 1.27)))
+    )
+    (property "Footprint" "Resistor_SMD:R_0603_1608Metric_Pad0.98x0.95mm_HandSolder" (at 181.102 115.57 0)
+      (effects (font (size 1.27 1.27)) hide)
+    )
+    (property "Datasheet" "~" (at 181.102 115.57 0)
+      (effects (font (size 1.27 1.27)) hide)
+    )
